File: hw/EAGLE/Prototyping/Tiny841/Tiny841.brd (EAGLE design)
At the start: 160 x 100 mm, 10 parts, among them IC1 ATTINY44-SSU

Commit message: added full 841 board
Parts:
- added C1: (no value), SparkFun-Capacitors:PANASONIC_D
- added C2: CAP-UNPOLARIZEDFAB, fab:C1206FAB
- added J6: (no value), SparkFun-Connectors:1X02
- added U$1: ACS712, SparkFun-AnalogIC:SO08
- J5: device SparkFun-Connectors:1X02 -> SparkFun-Connectors:SCREWTERMINAL-3.5MM-2-NS
- moved J5 82.3 mm to (44.7, 57.9), turned to 270 degrees
- moved R1 71.0 mm to (61.0, 34.8), turned to 90 degrees
- moved R2 68.6 mm to (61.0, 26.2), turned to 270 degrees
- moved J4 66.3 mm to (66.0, 38.5), turned to 180 degrees
- moved U$2 49.2 mm to (47.8, 41.9)
- moved J3 49.1 mm to (48.9, 29.1)
- moved J2 49.1 mm to (46.4, 29.1)
- moved J1 48.8 mm to (56.1, 45.3)
- moved U$3 47.8 mm to (55.4, 30.5), turned to 270 degrees
- moved IC1 47.7 mm to (54.9, 39.2)
Connections:
- new net N$8: C2.1, U$1.6
- new net VCC_RAW: C1.+, J5.2, U$1.1, U$1.2, U$1.8
- net CURSENSE: now also U$1.7; no longer J5.2
- net GND: now also C1.-, C2.2, U$1.5
- net SCL: now also J6.1
- net SDA: now also J6.2
- net VCC: now also U$1.3, U$1.4
Routing:
- net GND: track 0.00 -> 53.4 mm, vias 0 -> 4
- net SDA: track 0.00 -> 22.7 mm
- net CURSENSE: track 0.00 -> 18.3 mm
- net SCL: track 0.00 -> 18.1 mm
- net MOTSIG0: track 0.00 -> 9.72 mm
- net MOTSIG2: track 0.00 -> 9.40 mm
- net RESET: track 0.00 -> 9.33 mm
- net N$6: track 0.00 -> 5.99 mm
- net MOTSIG1: track 0.00 -> 5.91 mm
- net VCC_RAW: track 0.00 -> 5.23 mm
- net N$5: track 0.00 -> 4.77 mm
- net N$8: track 0.00 -> 3.13 mm
- added copper zone on layer 1, net GND
- added copper zone on layer 1, net VCC
- added copper zone on layer 1, net VCC_RAW
Other:
- board size 160 x 100 mm -> 29.2 x 38.5 mm
