File: hw/EAGLE/Prototyping/Tiny841/Tiny841.sch (EAGLE design)
At the start: 10 parts, among them IC1 ATTINY44-SSU

Commit message: added full 841 board
Parts:
- added C1: (no value), SparkFun-Capacitors:47UF-50V-20%(ELECT)
- added C2: CAP-UNPOLARIZEDFAB, fab:CAP-UNPOLARIZEDFAB
- added J6: (no value), SparkFun-Connectors:M02PTH
- added U$1: ACS712, SparkFun-AnalogIC:ACS712
- J5: device SparkFun-Connectors:M02PTH -> SparkFun-Connectors:M023.5MM-NO_SILK
Connections:
- new net N$8: C2.1, U$1.FILT
- new net VCC_RAW: C1.+, J5.2, U$1.IP+@1, U$1.IP+@2, U$1.VCC
- net CURSENSE: now also U$1.VOUT; no longer J5.2
- net GND: now also C1.-, C2.2, U$1.GND
- net SCL: now also J6.1
- net SDA: now also J6.2
- net VCC: now also U$1.IP-@3, U$1.IP-@4
Other:
- moved on the sheet: J5
Changed lines of the file:
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@@
 <?xml version="1.0" encoding="utf-8"?>
 <!DOCTYPE eagle SYSTEM "eagle.dtd">
-<eagle version="7.4.0">
+<eagle version="7.2.0">
 <drawing>
 <settings>
@@
 <part name="R1" library="fab" deviceset="RES-US" device="1206FAB"/>
 <part name="R2" library="fab" deviceset="RES-US" device="1206FAB"/>
-<part name="J5" library="SparkFun-Connectors" deviceset="M02" device="PTH"/>
+<part name="U$1" library="SparkFun-AnalogIC" deviceset="ACS712" device=""/>
+<part name="J5" library="SparkFun-Connectors" deviceset="M02" device="3.5MM-NO_SILK"/>
+<part name="GND6" library="SparkFun-Aesthetics" deviceset="GND" device=""/>
+<part name="C1" library="SparkFun-Capacitors" deviceset="47UF-50V-20%(ELECT)" device=""/>
+<part name="GND5" library="SparkFun-Aesthetics" deviceset="GND" device=""/>
+<part name="C2" library="fab" deviceset="CAP-UNPOLARIZED" device="FAB"/>
+<part name="J6" library="SparkFun-Connectors" deviceset="M02" device="PTH"/>
 </parts>
 <sheets>
@@
 <instance part="R1" gate="G$1" x="127" y="147.32" rot="R90"/>
 <instance part="R2" gate="G$1" x="142.24" y="147.32" rot="R90"/>
-<instance part="J5" gate="G$1" x="-20.32" y="109.22"/>
+<instance part="U$1" gate="G$1" x="203.2" y="172.72"/>
+<instance part="J5" gate="G$1" x="129.54" y="175.26"/>
+<instance part="GND6" gate="1" x="226.06" y="154.94"/>
+<instance part="C1" gate="G$1" x="147.32" y="172.72"/>
+<instance part="GND5" gate="1" x="139.7" y="160.02"/>
+<instance part="C2" gate="&gt;NAME" x="233.68" y="165.1" rot="R270"/>
+<instance part="J6" gate="G$1" x="63.5" y="68.58"/>
 </instances>
 <busses>
@@
 <label x="129.54" y="137.16" size="1.778" layer="95"/>
 </segment>
+<segment>
+<pinref part="J6" gate="G$1" pin="2"/>
+<wire x1="71.12" y1="71.12" x2="88.9" y2="71.12" width="0.1524" layer="91"/>
+</segment>
 </net>
 <net name="MOTSIG2" class="0">
@@
 <label x="114.3" y="137.16" size="1.778" layer="95"/>
 </segment>
+<segment>
+<pinref part="J6" gate="G$1" pin="1"/>
+<wire x1="71.12" y1="68.58" x2="88.9" y2="68.58" width="0.1524" layer="91"/>
+</segment>
 </net>
 <net name="CURSENSE" class="0">
@@
 </segment>
 <segment>
-<pinref part="J5" gate="G$1" pin="2"/>
-<wire x1="-12.7" y1="111.76" x2="-2.54" y2="111.76" width="0.1524" layer="91"/>
-<label x="-10.16" y="111.76" size="1.778" layer="95"/>
+<pinref part="U$1" gate="G$1" pin="VOUT"/>
+<wire x1="215.9" y1="175.26" x2="238.76" y2="175.26" width="0.1524" layer="91"/>
+<label x="231.14" y="175.26" size="1.778" layer="95"/>
 </segment>
 </net>
@@
 <label x="142.24" y="152.4" size="1.778" layer="95" rot="R90"/>
 </segment>
+<segment>
+<pinref part="U$1" gate="G$1" pin="IP-@4"/>
+<wire x1="187.96" y1="170.18" x2="182.88" y2="170.18" width="0.1524" layer="91"/>
+<pinref part="U$1" gate="G$1" pin="IP-@3"/>
+<wire x1="182.88" y1="170.18" x2="167.64" y2="170.18" width="0.1524" layer="91"/>
+<wire x1="187.96" y1="172.72" x2="182.88" y2="172.72" width="0.1524" layer="91"/>
+<wire x1="182.88" y1="172.72" x2="182.88" y2="170.18" width="0.1524" layer="91"/>
+<label x="170.18" y="170.18" size="1.778" layer="95"/>
+</segment>
 </net>
 <net name="GND" class="0">
@@
 <wire x1="12.7" y1="104.14" x2="12.7" y2="101.6" width="0.1524" layer="91"/>
 <junction x="12.7" y="104.14"/>
+</segment>
+<segment>
+<pinref part="U$1" gate="G$1" pin="GND"/>
+<wire x1="215.9" y1="170.18" x2="226.06" y2="170.18" width="0.1524" layer="91"/>
+<wire x1="226.06" y1="170.18" x2="226.06" y2="160.02" width="0.1524" layer="91"/>
+<pinref part="GND6" gate="1" pin="GND"/>
+<pinref part="C2" gate="&gt;NAME" pin="2"/>
+<wire x1="226.06" y1="160.02" x2="226.06" y2="157.48" width="0.1524" layer="91"/>
+<wire x1="233.68" y1="162.56" x2="233.68" y2="160.02" width="0.1524" layer="91"/>
+<wire x1="233.68" y1="160.02" x2="226.06" y2="160.02" width="0.1524" layer="91"/>
+<junction x="226.06" y="160.02"/>
+</segment>
+<segment>
 <pinref part="J5" gate="G$1" pin="1"/>
-<wire x1="-12.7" y1="109.22" x2="-7.62" y2="109.22" width="0.1524" layer="91"/>
-<wire x1="-7.62" y1="109.22" x2="-7.62" y2="104.14" width="0.1524" layer="91"/>
-<wire x1="-7.62" y1="104.14" x2="12.7" y2="104.14" width="0.1524" layer="91"/>
+<wire x1="137.16" y1="175.26" x2="139.7" y2="175.26" width="0.1524" layer="91"/>
+<wire x1="139.7" y1="175.26" x2="139.7" y2="165.1" width="0.1524" layer="91"/>
+<pinref part="C1" gate="G$1" pin="-"/>
+<wire x1="147.32" y1="167.64" x2="147.32" y2="165.1" width="0.1524" layer="91"/>
+<wire x1="147.32" y1="165.1" x2="139.7" y2="165.1" width="0.1524" layer="91"/>
+<wire x1="139.7" y1="165.1" x2="139.7" y2="162.56" width="0.1524" layer="91"/>
+<pinref part="GND5" gate="1" pin="GND"/>
 </segment>
 </net>
@@
 </segment>
 </net>
+<net name="VCC_RAW" class="0">
+<segment>
+<pinref part="U$1" gate="G$1" pin="IP+@1"/>
+<wire x1="187.96" y1="177.8" x2="182.88" y2="177.8" width="0.1524" layer="91"/>
+<pinref part="U$1" gate="G$1" pin="IP+@2"/>
+<wire x1="187.96" y1="175.26" x2="182.88" y2="175.26" width="0.1524" layer="91"/>
+<wire x1="182.88" y1="175.26" x2="182.88" y2="177.8" width="0.1524" layer="91"/>
+<pinref part="J5" gate="G$1" pin="2"/>
+<wire x1="137.16" y1="177.8" x2="147.32" y2="177.8" width="0.1524" layer="91"/>
+<pinref part="C1" gate="G$1" pin="+"/>
+<wire x1="147.32" y1="177.8" x2="182.88" y2="177.8" width="0.1524" layer="91"/>
+<wire x1="147.32" y1="175.26" x2="147.32" y2="177.8" width="0.1524" layer="91"/>
+<junction x="147.32" y="177.8"/>
+<label x="167.64" y="177.8" size="1.778" layer="95"/>
+</segment>
+<segment>
+<pinref part="U$1" gate="G$1" pin="VCC"/>
+<wire x1="215.9" y1="177.8" x2="226.06" y2="177.8" width="0.1524" layer="91"/>
+<wire x1="226.06" y1="177.8" x2="226.06" y2="190.5" width="0.1524" layer="91"/>
+<label x="226.06" y="185.42" size="1.778" layer="95" rot="R90"/>
+</segment>
+</net>
+<net name="N$8" class="0">
+<segment>
+<pinref part="U$1" gate="G$1" pin="FILT"/>
+<wire x1="215.9" y1="172.72" x2="233.68" y2="172.72" width="0.1524" layer="91"/>
+<pinref part="C2" gate="&gt;NAME" pin="1"/>
+<wire x1="233.68" y1="172.72" x2="233.68" y2="170.18" width="0.1524" layer="91"/>
+</segment>
+</net>
