File: hw/PCB/KICAD/R21_Core/R21_Core.sch (KiCad schematic (older format))
At the start: 96 parts, among them J1 JTAGICE3-10p, Q1 MOSFET_N, SW1 SPST_SW, T1 TPS61089RNR, U1 SAMR21E, U10 USB2, U11 AP2112K, U2 AP2112K, U3 LSM9DS1, U4 TPS2559-Q1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

Commit message: Lots of changes- firmware, board rev, mods
Connections:
- net BB_GND: now also D2.1, D3.1; no longer D2.2, D3.2
- net GND: now also D1.1; no longer D1.2
- net at R1.1: now also D1.2; no longer D1.1
- net at Q1.D: now also D5.1; no longer D5.2
- net at R12.1: now also D5.2; no longer D5.1
- net at R9.1: now also D3.2; no longer D3.1
- net at R2.1: now also D2.2; no longer D2.1
Changed lines of the file:
@@
 F 3 "" H 3650 1625 60  0001 C CNN
 	1    3650 1600
-	-1   0    0    1
+	1    0    0    -1
 $EndComp
 $Comp
@@
 F 3 "" H 4000 1625 60  0001 C CNN
 	1    4000 1600
-	-1   0    0    1
+	1    0    0    -1
 $EndComp
 $Comp
@@
 F 3 "" H 12600 5925 60  0001 C CNN
 	1    12600 5900
-	-1   0    0    1
+	1    0    0    -1
 $EndComp
 Text GLabel 12600 5500 1    39   Input ~ 0
@@
 F 3 "" H 12350 5925 60  0001 C CNN
 	1    12350 5900
-	-1   0    0    1
-$EndComp
-$Comp
+	1    0    0    -1
+$EndComp
+$Comp

Commit message: Added addendum to boards, modules for debug, comms description
Connections:
- net BB_SCL: now also U5.5 (A0)
Changed lines of the file:
@@
 Wire Wire Line
 	2950 -1550 2900 -1550
+Wire Wire Line
+	10200 1150 10250 1150
+Wire Wire Line
+	10250 1150 10250 1100
+Connection ~ 10250 1100
 $EndSCHEMATC
